File: hardware/brd/smartcane.brd (EAGLE design)
At the start: 68.6 x 53.3 mm, 5 parts

Commit message: Documentacao + codigo + circuito
Parts:
- removed K3: (no value), AUTODESK_CIRCUITS_BREADBOARD:M3XXH
- removed R1: 1k‎Ω, AUTODESK_CIRCUITS_BREADBOARD:0207/10
Connections:
- removed net N$1 (its old number): PING2.3, U1.5
- removed net N$5: K3.O
- removed net N$6: K3.S, M1.2
- removed net N$7: K3.P
- removed net N$8: K3.2, R1.1, R1.2, U1.13
- new net N$2: M1.1, PING2.1, U1.GND..
- net N$3: now also PING2.3, U1.6; no longer K3.P@
- net N$4: now also M1.2, U1.11; no longer K3.1, M1.1, PING2.1, U1.GND..
Changed lines of the file:
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@@
 </autorouter>
 <elements>
-<element value="" name="U1" library="AUTODESK_CIRCUITS_BREADBOARD" package="ARDUINO_UNO" x="5" y="10.08"></element><element value="" name="PING2" library="AUTODESK_CIRCUITS_BREADBOARD" package="1X3P-2.54-2.54-11.6-3.0-BLACK-MALE" x="5" y="22.78"></element><element value="" name="M1" library="AUTODESK_CIRCUITS_BREADBOARD" package="2P-2.54-65/35MIL" x="5" y="35.480000000000004"></element><element value="" name="K3" library="AUTODESK_CIRCUITS_BREADBOARD" package="M3XXH" x="5" y="48.18"></element><element value="1k‎Ω" name="R1" library="AUTODESK_CIRCUITS_BREADBOARD" package="0207/10" x="5" y="60.879999999999995"></element></elements>
+<element value="" name="U1" library="AUTODESK_CIRCUITS_BREADBOARD" package="ARDUINO_UNO" x="5" y="10.08"></element><element value="" name="PING2" library="AUTODESK_CIRCUITS_BREADBOARD" package="1X3P-2.54-2.54-11.6-3.0-BLACK-MALE" x="5" y="22.78"></element><element value="" name="M1" library="AUTODESK_CIRCUITS_BREADBOARD" package="2P-2.54-65/35MIL" x="5" y="35.480000000000004"></element></elements>
 <signals>
-<signal name="N$1"><contactref element="U1" pad="5"></contactref><contactref element="PING2" pad="3"></contactref><wire x1="55.8" y1="60.879999999999995" x2="5" y2="20.240000000000002" width="0" layer="19" extent="1-1"></wire></signal><signal name="N$2"><contactref element="PING2" pad="2"></contactref><contactref element="U1" pad="5V"></contactref><wire x1="5" y1="22.78" x2="43.1" y2="12.620000000000001" width="0" layer="19" extent="1-1"></wire></signal><signal name="N$3"><contactref element="K3" pad="P@"></contactref></signal><signal name="N$4"><contactref element="K3" pad="1"></contactref><contactref element="PING2" pad="1"></contactref><wire x1="1.19" y1="51.99" x2="5" y2="25.32" width="0" layer="19" extent="1-1"></wire><contactref element="U1" pad="GND.."></contactref><wire x1="5" y1="25.32" x2="45.64" y2="12.620000000000001" width="0" layer="19" extent="1-1"></wire><contactref element="M1" pad="1"></contactref><wire x1="45.64" y1="12.620000000000001" x2="5" y2="36.75000000000001" width="0" layer="19" extent="1-1"></wire></signal><signal name="N$5"><contactref element="K3" pad="O"></contactref></signal><signal name="N$6"><contactref element="K3" pad="S"></contactref><contactref element="M1" pad="2"></contactref><wire x1="-1.3499999999999996" y1="51.99" x2="5" y2="34.21" width="0" layer="19" extent="1-1"></wire></signal><signal name="N$7"><contactref element="K3" pad="P"></contactref></signal><signal name="N$8"><contactref element="R1" pad="1"></contactref><contactref element="U1" pad="13"></contactref><wire x1="-0.08000000000000007" y1="60.879999999999995" x2="33.956" y2="60.879999999999995" width="0" layer="19" extent="1-1"></wire><contactref element="K3" pad="2"></contactref><wire x1="33.956" y1="60.879999999999995" x2="1.19" y2="44.37" width="0" layer="19" extent="1-1"></wire><contactref element="R1" pad="2"></contactref><wire x1="1.19" y1="44.37" x2="10.08" y2="60.879999999999995" width="0" layer="19" extent="1-1"></wire></signal></signals>
+<signal name="N$1"><contactref element="U1" pad="5V"></contactref><contactref element="PING2" pad="2"></contactref><wire x1="43.1" y1="12.620000000000001" x2="5" y2="22.78" width="0" layer="19" extent="1-1"></wire></signal><signal name="N$2"><contactref element="U1" pad="GND.."></contactref><contactref element="M1" pad="1"></contactref><wire x1="45.64" y1="12.620000000000001" x2="5" y2="36.75000000000001" width="0" layer="19" extent="1-1"></wire><contactref element="PING2" pad="1"></contactref><wire x1="5" y1="36.75000000000001" x2="5" y2="25.32" width="0" layer="19" extent="1-1"></wire></signal><signal name="N$3"><contactref element="U1" pad="6"></contactref><contactref element="PING2" pad="3"></contactref><wire x1="53.26" y1="60.879999999999995" x2="5" y2="20.240000000000002" width="0" layer="19" extent="1-1"></wire></signal><signal name="N$4"><contactref element="M1" pad="2"></contactref><contactref element="U1" pad="11"></contactref><wire x1="5" y1="34.21" x2="39.036" y2="60.879999999999995" width="0" layer="19" extent="1-1"></wire></signal></signals>
 </board>
 </drawing>
